Commit message: Added laser Scan (360), made laser_sensor link length=0.15 , sensror at position= 0.13

File: urdf/robot_description.urdf.xacro (robot description, xacro)
@@ -44,12 +44,12 @@
       </surface>
     </collision>
-    <!-- <visual name="$(arg robot_name)/caster_front_visual">
+    <visual name="$(arg robot_name)/caster_front_visual">
       <origin rpy=" 0 0 0" xyz="0.2 0 -0.05"/>
       <geometry>
         <sphere radius="0.05"/>
       </geometry>
-    </visual> -->
+    </visual>
   </link>
-  <link name="$(arg robot_name)/sensor_ir">
+  <link name="$(arg robot_name)/sensor_laser">
     <inertial>
         <origin xyz="0 0 0" rpy="0 0 0" />
@@ -60,19 +60,19 @@
         <origin xyz="0 0 0" rpy="0 0 0" />
         <geometry>
-        <cylinder radius="0.05" length="0.1"/>
+        <cylinder radius="0.05" length="0.15"/>
         </geometry>
         <material name="white" />
     </visual>
-       <!-- <collision>
+       <collision>
         <origin xyz="0 0 0" rpy="0 0 0"/>
         <geometry>
-        <cylinder radius="0.05" length="0.1"/>
+        <cylinder radius="0.05" length="0.15"/>
         </geometry>
-    </collision> -->
+    </collision>
   </link>
-  <joint name="$(arg robot_name)/joint_sensor_ir" type="fixed">
-    <origin xyz="0.15 0 0.05" rpy="0 0 0"/>
+  <joint name="$(arg robot_name)/joint_sensor_laser" type="fixed">
+    <origin xyz="0.15 0 0.13" rpy="0 0 0"/>
     <parent link="$(arg robot_name)/link_chassis"/>
-    <child link="$(arg robot_name)/sensor_ir"/>
+    <child link="$(arg robot_name)/sensor_laser"/>
   </joint>
   <xacro:link_wheel name="$(arg robot_name)/link_right_wheel" />

Commit message: changed the go2goal controller.Seems to go to the closest point.Pops the tf_buffer/laser atribute error sometimes.

File: urdf/robot_description.urdf.xacro (robot description, xacro)
@@ -11,5 +11,6 @@
     <inertial>
       <mass value="5"/>
-      <origin rpy="0 0 0" xyz="0 0 0.1"/>
+      <!-- z=0.1 -->
+      <origin rpy="0 0 0" xyz="0 0 0"/>
       <inertia ixx="0.0395416666667" ixy="0" ixz="0" iyy="0.106208333333" iyz="0" izz="0.106208333333"/>
     </inertial>
@@ -64,5 +65,5 @@
         <material name="white" />
     </visual>
-       <collision>
+    <collision>
         <origin xyz="0 0 0" rpy="0 0 0"/>
         <geometry>

Commit message: changed location of sensor joint on URDF and the field of vision of the robot

File: urdf/robot_description.urdf.xacro (robot description, xacro)
@@ -73,5 +73,5 @@
   </link>
   <joint name="$(arg robot_name)/joint_sensor_laser" type="fixed">
-    <origin xyz="0.15 0 0.13" rpy="0 0 0"/>
+    <origin xyz="0 0 0.13" rpy="0 0 0"/>
     <parent link="$(arg robot_name)/link_chassis"/>
     <child link="$(arg robot_name)/sensor_laser"/>
