Commit message: Add files via upload

File: urdf/macros.xacro (robot description, xacro)
@@ -1,6 +1,6 @@
 <?xml version="1.0"?>
-<robot>
-	<macro name="link_wheel" params="name">
-		<link name="${name}">
+<robot xmlns:xacro="http://wiki.ros.org/xacro">
+	<xacro:macro name="link_wheel" params="robot">
+		<link name="${robot}_link_wheel">
 		    <inertial>
 		      <mass value="0.2"/>
@@ -8,5 +8,5 @@
 		      <inertia ixx="0.000526666666667" ixy="0" ixz="0" iyy="0.000526666666667" iyz="0" izz="0.001"/>
 		    </inertial>
-		    <collision name="${name}_collision">
+		    <collision name="${robot}_collision">
 		      <origin rpy="0 1.5707 1.5707" xyz="0 0 0"/>
 		      <geometry>
@@ -14,5 +14,5 @@
 		      </geometry>
 		    </collision>
-		    <visual name="${name}_visual">
+		    <visual name="${robot}_visual">
 		      <origin rpy="0 1.5707 1.5707" xyz="0 0 0"/>
 		      <geometry>
@@ -21,4 +21,4 @@
 		    </visual>
 		  </link>
-	</macro>
+	</xacro:macro>
 </robot>

File: urdf/robot_description.urdf.xacro (robot description, xacro)
@@ -3,7 +3,7 @@
   <xacro:arg name="robot_name" default="robot"/>
 <!--  -->
-<xacro:include filename="$(find swarm)/urdf/materials.xacro"/>
-<xacro:include filename="$(find swarm)/urdf/robot_gazebo_plugins.gazebo"/>
-<xacro:include filename="$(find swarm)/urdf/macros.xacro"/>
+	<xacro:include filename="$(find swarm)/urdf/materials.xacro"/>
+	<xacro:include filename="$(find swarm)/urdf/robot_gazebo_plugins.gazebo"/>
+	<xacro:include filename="$(find swarm)/urdf/macros.xacro"/>
   <link name="$(arg robot_name)/link_chassis">
     <!-- pose and inertia -->
@@ -77,5 +77,25 @@
     <child link="$(arg robot_name)/sensor_laser"/>
   </joint>
-  <xacro:link_wheel name="$(arg robot_name)/link_right_wheel" />
+<!--   <xacro:link_wheel name="$(arg robot_name)/link_right_wheel" />
+ -->
+	<link name="$(arg robot_name)/link_right_wheel">
+		    <inertial>
+		      <mass value="0.2"/>
+		      <origin rpy="0 1.5707 1.5707" xyz="0 0 0"/>
+		      <inertia ixx="0.000526666666667" ixy="0" ixz="0" iyy="0.000526666666667" iyz="0" izz="0.001"/>
+		    </inertial>
+		    <collision name="$(arg robot_name)/link_right_wheel_collision">
+		      <origin rpy="0 1.5707 1.5707" xyz="0 0 0"/>
+		      <geometry>
+		        <cylinder length="0.04" radius="0.1"/>
+		      </geometry>
+		    </collision>
+		    <visual name="$(arg robot_name)/link_right_wheel_visual">
+		      <origin rpy="0 1.5707 1.5707" xyz="0 0 0"/>
+		      <geometry>
+		        <cylinder length="0.04" radius="0.1"/>
+		      </geometry>
+		    </visual>
+		  </link>
   <joint name="$(arg robot_name)/joint_right_wheel" type="continuous">
     <origin rpy="0 0 0" xyz="-0.05 0.15 0"/>
@@ -86,5 +106,24 @@
     <joint_properties damping="1.0" friction="1.0"/>
   </joint>
-  <xacro:link_wheel name="$(arg robot_name)/link_left_wheel" />
+<!--  <xacro:link_wheel name="$(arg robot_name)/link_left_wheel" />
+ -->	<link name="$(arg robot_name)/link_left_wheel">
+		    <inertial>
+		      <mass value="0.2"/>
+		      <origin rpy="0 1.5707 1.5707" xyz="0 0 0"/>
+		      <inertia ixx="0.000526666666667" ixy="0" ixz="0" iyy="0.000526666666667" iyz="0" izz="0.001"/>
+		    </inertial>
+		    <collision name="$(arg robot_name)/link_left_wheel_collision">
+		      <origin rpy="0 1.5707 1.5707" xyz="0 0 0"/>
+		      <geometry>
+		        <cylinder length="0.04" radius="0.1"/>
+		      </geometry>
+		    </collision>
+		    <visual name="$(arg robot_name)/link_left_wheel_visual">
+		      <origin rpy="0 1.5707 1.5707" xyz="0 0 0"/>
+		      <geometry>
+		        <cylinder length="0.04" radius="0.1"/>
+		      </geometry>
+		    </visual>
+		  </link>
   <joint name="$(arg robot_name)/joint_left_wheel" type="continuous">
     <origin rpy="0 0 0" xyz="-0.05 -0.15 0"/>
